Commit message: Removed the mimic element from the finger joint2

File: franka_description/robots/hand.xacro (robot description, xacro)
@@ -71,5 +71,4 @@
       <axis xyz="0 -1 0"/>
       <limit effort="20" lower="0.0" upper="0.04" velocity="0.2"/>
-      <mimic joint="${ns}_finger_joint1" />
     </joint>
   </xacro:macro>
